Commit message: added caster wheels and optimized kinematic parameters

File: src/outr_description/urdf/outr.xacro (robot description, xacro)
@@ -1,19 +1,17 @@
 <?xml version='1.0'?>
-<robot name="robot" xmlns:xacro="http://www.ros.org/wiki/xacro">
+<robot name="robot"
+  xmlns:xacro="http://www.ros.org/wiki/xacro">
   <xacro:include filename="$(find outr_description)/urdf/outr.gazebo" />
   <xacro:include filename="$(find outr_description)/urdf/materials.xacro" />
   <xacro:include filename="$(find outr_description)/urdf/macros.xacro" />
   <link name='chassis'>
-    <pose>0 0 0.1 0 0 0</pose>
+    <pose>0 0 0 0 0 0</pose>
     <inertial>
       <mass value="10.0"/>
-      <origin xyz="0.0 0 0.1" rpy=" 0 0 0"/>
-      <inertia
-          ixx="0.5" ixy="0" ixz="0"
-          iyy="1.0" iyz="0"
-          izz="0.1"
-      />
+      <origin xyz="0.15 0 -0.1" rpy=" 0 0 3.14159"/>
+      <inertia ixx="0.5" ixy="0" ixz="0" iyy="1.0" iyz="0" izz="0.5" />
     </inertial>
     <collision name='collision'>
+      <origin xyz="0.15 0 -0.1" rpy=" 0 0 3.14159"/>
       <geometry>
         <mesh filename="package://outr_description/urdf/outr.dae"/>
@@ -21,27 +19,93 @@
     </collision>
     <visual name='chassis_visual'>
-      <origin xyz="0 0 0" rpy=" 0 0 0"/>
+      <origin xyz="0.15 0 -0.1" rpy=" 0 0 3.14159"/>
       <geometry>
         <mesh filename="package://outr_description/urdf/outr.dae"/>
       </geometry>
     </visual>
-    <collision name='caster_collision'>
-      <origin xyz="-0.15 0 -0.05" rpy=" 0 0 0"/>
-      <geometry>
-        <sphere radius="0.05"/>
-      </geometry>
-      <surface>
-        <friction>
-          <ode>
-            <mu>0</mu>
-            <mu2>0</mu2>
-            <slip1>1.0</slip1>
-            <slip2>1.0</slip2>
-          </ode>
-        </friction>
-      </surface>
-    </collision>
-    <visual name='caster_visual'>
-      <origin xyz="-0.15 0 -0.05" rpy=" 0 0 0"/>
+    <collision name='caster1_collision'>
+      <origin xyz="0.45 0.22 -0.04" rpy=" 0 0 0"/>
+      <geometry>
+        <sphere radius="0.05"/>
+      </geometry>
+      <surface>
+        <friction>
+          <ode>
+            <mu>0</mu>
+            <mu2>0</mu2>
+            <slip1>5.0</slip1>
+            <slip2>5.0</slip2>
+          </ode>
+        </friction>
+      </surface>
+    </collision>
+    <visual name='caster1_visual'>
+      <origin xyz="0.45 0.22 -0.04" rpy=" 0 0 0"/>
+      <geometry>
+        <sphere radius="0.05"/>
+      </geometry>
+    </visual>
+    <collision name='caster2_collision'>
+      <origin xyz="0.45 -0.22 -0.04" rpy=" 0 0 0"/>
+      <geometry>
+        <sphere radius="0.05"/>
+      </geometry>
+      <surface>
+        <friction>
+          <ode>
+            <mu>0</mu>
+            <mu2>0</mu2>
+            <slip1>5.0</slip1>
+            <slip2>5.0</slip2>
+          </ode>
+        </friction>
+      </surface>
+    </collision>
+    <visual name='caster2_visual'>
+      <origin xyz="0.45 -0.22 -0.04" rpy=" 0 0 0"/>
+      <geometry>
+        <sphere radius="0.05"/>
+      </geometry>
+    </visual>
+    <collision name='caster3_collision'>
+      <origin xyz="-0.45 0.22 -0.04" rpy=" 0 0 0"/>
+      <geometry>
+        <sphere radius="0.05"/>
+      </geometry>
+      <surface>
+        <friction>
+          <ode>
+            <mu>0</mu>
+            <mu2>0</mu2>
+            <slip1>5.0</slip1>
+            <slip2>5.0</slip2>
+          </ode>
+        </friction>
+      </surface>
+    </collision>
+    <visual name='caster3_visual'>
+      <origin xyz="-0.45 0.22 -0.04" rpy=" 0 0 0"/>
+      <geometry>
+        <sphere radius="0.05"/>
+      </geometry>
+    </visual>
+    <collision name='caster4_collision'>
+      <origin xyz="-0.45 -0.22 -0.04" rpy=" 0 0 0"/>
+      <geometry>
+        <sphere radius="0.05"/>
+      </geometry>
+      <surface>
+        <friction>
+          <ode>
+            <mu>0</mu>
+            <mu2>0</mu2>
+            <slip1>5.0</slip1>
+            <slip2>5.0</slip2>
+          </ode>
+        </friction>
+      </surface>
+    </collision>
+    <visual name='caster4_visual'>
+      <origin xyz="-0.45 -0.22 -0.04" rpy=" 0 0 0"/>
       <geometry>
         <sphere radius="0.05"/>
@@ -50,15 +114,29 @@
   </link>
   <link name="left_wheel">
-    <!--origin xyz="0.1 0.13 0.1" rpy="0 1.5707 1.5707"/-->
     <collision name="collision">
       <origin xyz="0 0 0" rpy="0 1.5707 1.5707"/>
       <geometry>
-        <cylinder radius="0.1" length="0.05"/>
-      </geometry>
+        <cylinder radius="0.1" length="0.03"/>
+      </geometry>
+      <surface>
+        <!-- <friction>
+          <ode>
+            <mu>5</mu>
+            <mu2>5</mu2>
+            <slip1>0</slip1>
+            <slip2>0</slip2>
+          </ode>
+        </friction> -->
+        <contact>
+          <ode>
+            <min_depth>5</min_depth>
+          </ode>
+        </contact>
+      </surface>
     </collision>
     <visual name="left_wheel_visual">
       <origin xyz="0 0 0" rpy="0 1.5707 1.5707"/>
       <geometry>
-        <cylinder radius="0.1" length="0.05"/>
+        <cylinder radius="0.1" length="0.03"/>
       </geometry>
     </visual>
@@ -66,23 +144,34 @@
       <origin xyz="0 0 0" rpy="0 1.5707 1.5707"/>
       <mass value="5"/>
-      <cylinder_inertia m="5" r="0.1" h="0.05"/>
-      <inertia
-        ixx="1.0" ixy="0.0" ixz="0.0"
-        iyy="1.0" iyz="0.0"
-        izz="1.0"/>
+      <cylinder_inertia m="5" r="0.1" h="0.03"/>
+      <inertia ixx="1.0" ixy="0.0" ixz="0.0" iyy="1.0" iyz="0.0" izz="1.0"/>
     </inertial>
   </link>
   <link name="right_wheel">
-    <!--origin xyz="0.1 -0.13 0.1" rpy="0 1.5707 1.5707"/-->
     <collision name="collision">
       <origin xyz="0 0 0" rpy="0 1.5707 1.5707"/>
       <geometry>
-        <cylinder radius="0.1" length="0.05"/>
-      </geometry>
+        <cylinder radius="0.1" length="0.03"/>
+      </geometry>
+      <surface>
+        <!-- <friction>
+          <ode>
+            <mu>5</mu>
+            <mu2>5</mu2>
+            <slip1>0</slip1>
+            <slip2>0</slip2>
+          </ode>
+        </friction> -->
+        <contact>
+          <ode>
+            <min_depth>5</min_depth>
+          </ode>
+        </contact>
+      </surface>
     </collision>
     <visual name="right_wheel_visual">
       <origin xyz="0 0 0" rpy="0 1.5707 1.5707"/>
       <geometry>
-        <cylinder radius="0.1" length="0.05"/>
+        <cylinder radius="0.1" length="0.03"/>
       </geometry>
     </visual>
@@ -90,25 +179,28 @@
       <origin xyz="0 0 0" rpy="0 1.5707 1.5707"/>
       <mass value="5"/>
-      <cylinder_inertia m="5" r="0.1" h="0.05"/>
-      <inertia
-        ixx="1.0" ixy="0.0" ixz="0.0"
-        iyy="1.0" iyz="0.0"
-        izz="1.0"/>
+      <cylinder_inertia m="5" r="0.1" h="0.03"/>
+      <inertia ixx="1.0" ixy="0.0" ixz="0.0" iyy="1.0" iyz="0.0" izz="1.0"/>
     </inertial>
   </link>
+  <gazebo reference="right_wheel">
+    <material>WheelMaterial</material>
+  </gazebo>
+  <gazebo reference="left_wheel">
+    <material>WheelMaterial</material>
+  </gazebo>
   <joint type="continuous" name="left_wheel_hinge">
-    <origin xyz="0.1 0.15 0" rpy="0 0 0"/>
+    <origin xyz="0 0.22 0" rpy="0 0 0"/>
     <child link="left_wheel"/>
     <parent link="chassis"/>
     <axis xyz="0 1 0" rpy="0 0 0"/>
-    <limit effort="100" velocity="100"/>
+    <limit effort="100000000" velocity="100000000"/>
     <joint_properties damping="0.0" friction="0.0"/>
   </joint>
   <joint type="continuous" name="right_wheel_hinge">
-    <origin xyz="0.1 -0.15 0" rpy="0 0 0"/>
+    <origin xyz="0 -0.22 0" rpy="0 0 0"/>
     <child link="right_wheel"/>
     <parent link="chassis"/>
     <axis xyz="0 1 0" rpy="0 0 0"/>
-    <limit effort="100" velocity="100"/>
+    <limit effort="100000000" velocity="100000000"/>
     <joint_properties damping="0.0" friction="0.0"/>
   </joint>

Commit message: added laserscanner from pointcloud functionality, added new package for navigation stack, readme to be updated

File: src/outr_description/urdf/outr.xacro (robot description, xacro)
@@ -5,13 +5,14 @@
   <xacro:include filename="$(find outr_description)/urdf/materials.xacro" />
   <xacro:include filename="$(find outr_description)/urdf/macros.xacro" />
+  <xacro:include filename="$(find outr_description)/urdf/_d435.urdf.xacro"/>
   <link name='chassis'>
     <pose>0 0 0 0 0 0</pose>
     <inertial>
-      <mass value="10.0"/>
-      <origin xyz="0.15 0 -0.1" rpy=" 0 0 3.14159"/>
-      <inertia ixx="0.5" ixy="0" ixz="0" iyy="1.0" iyz="0" izz="0.5" />
+      <mass value="5.0"/>
+      <origin xyz="0.15 0 -0.15" rpy=" 0 0 3.14159"/>
+      <inertia ixx="100.0" ixy="0" ixz="0" iyy="100.0" iyz="0" izz="100.0" />
     </inertial>
     <collision name='collision'>
-      <origin xyz="0.15 0 -0.1" rpy=" 0 0 3.14159"/>
+      <origin xyz="0.15 0 -0.15" rpy=" 0 0 3.14159"/>
       <geometry>
         <mesh filename="package://outr_description/urdf/outr.dae"/>
@@ -19,5 +20,5 @@
     </collision>
     <visual name='chassis_visual'>
-      <origin xyz="0.15 0 -0.1" rpy=" 0 0 3.14159"/>
+      <origin xyz="0.15 0 -0.15" rpy=" 0 0 3.14159"/>
       <geometry>
         <mesh filename="package://outr_description/urdf/outr.dae"/>
@@ -25,5 +26,5 @@
     </visual>
     <collision name='caster1_collision'>
-      <origin xyz="0.45 0.22 -0.04" rpy=" 0 0 0"/>
+      <origin xyz="0.45 0.22 -0.05" rpy=" 0 0 0"/>
       <geometry>
         <sphere radius="0.05"/>
@@ -41,5 +42,5 @@
     </collision>
     <visual name='caster1_visual'>
-      <origin xyz="0.45 0.22 -0.04" rpy=" 0 0 0"/>
+      <origin xyz="0.45 0.22 -0.05" rpy=" 0 0 0"/>
       <geometry>
         <sphere radius="0.05"/>
@@ -47,5 +48,5 @@
     </visual>
     <collision name='caster2_collision'>
-      <origin xyz="0.45 -0.22 -0.04" rpy=" 0 0 0"/>
+      <origin xyz="0.45 -0.22 -0.05" rpy=" 0 0 0"/>
       <geometry>
         <sphere radius="0.05"/>
@@ -63,5 +64,5 @@
     </collision>
     <visual name='caster2_visual'>
-      <origin xyz="0.45 -0.22 -0.04" rpy=" 0 0 0"/>
+      <origin xyz="0.45 -0.22 -0.05" rpy=" 0 0 0"/>
       <geometry>
         <sphere radius="0.05"/>
@@ -69,5 +70,5 @@
     </visual>
     <collision name='caster3_collision'>
-      <origin xyz="-0.45 0.22 -0.04" rpy=" 0 0 0"/>
+      <origin xyz="-0.45 0.22 -0.05" rpy=" 0 0 0"/>
       <geometry>
         <sphere radius="0.05"/>
@@ -85,5 +86,5 @@
     </collision>
     <visual name='caster3_visual'>
-      <origin xyz="-0.45 0.22 -0.04" rpy=" 0 0 0"/>
+      <origin xyz="-0.45 0.22 -0.05" rpy=" 0 0 0"/>
       <geometry>
         <sphere radius="0.05"/>
@@ -91,5 +92,5 @@
     </visual>
     <collision name='caster4_collision'>
-      <origin xyz="-0.45 -0.22 -0.04" rpy=" 0 0 0"/>
+      <origin xyz="-0.45 -0.22 -0.05" rpy=" 0 0 0"/>
       <geometry>
         <sphere radius="0.05"/>
@@ -107,5 +108,5 @@
     </collision>
     <visual name='caster4_visual'>
-      <origin xyz="-0.45 -0.22 -0.04" rpy=" 0 0 0"/>
+      <origin xyz="-0.45 -0.22 -0.05" rpy=" 0 0 0"/>
       <geometry>
         <sphere radius="0.05"/>
@@ -120,15 +121,15 @@
       </geometry>
       <surface>
-        <!-- <friction>
-          <ode>
-            <mu>5</mu>
-            <mu2>5</mu2>
+        <friction>
+          <ode>
+            <mu>50</mu>
+            <mu2>50</mu2>
             <slip1>0</slip1>
             <slip2>0</slip2>
           </ode>
-        </friction> -->
+        </friction>
         <contact>
           <ode>
-            <min_depth>5</min_depth>
+            <min_depth>10</min_depth>
           </ode>
         </contact>
@@ -155,15 +156,15 @@
       </geometry>
       <surface>
-        <!-- <friction>
-          <ode>
-            <mu>5</mu>
-            <mu2>5</mu2>
+        <friction>
+          <ode>
+            <mu>50</mu>
+            <mu2>50</mu2>
             <slip1>0</slip1>
             <slip2>0</slip2>
           </ode>
-        </friction> -->
+        </friction>
         <contact>
           <ode>
-            <min_depth>5</min_depth>
+            <min_depth>10</min_depth>
           </ode>
         </contact>
@@ -205,3 +206,6 @@
     <joint_properties damping="0.0" friction="0.0"/>
   </joint>
+  <sensor_d435 parent="chassis">
+    <origin xyz="0.63 0 0" rpy="0 0 0"/>
+  </sensor_d435>
 </robot>

Commit message: added package

File: src/outr_description/urdf/outr.xacro (robot description, xacro)
@@ -6,10 +6,11 @@
   <xacro:include filename="$(find outr_description)/urdf/macros.xacro" />
   <xacro:include filename="$(find outr_description)/urdf/_d435.urdf.xacro"/>
+  <link name="base_link" />
   <link name='chassis'>
     <pose>0 0 0 0 0 0</pose>
     <inertial>
-      <mass value="5.0"/>
+      <mass value="10.0"/>
       <origin xyz="0.15 0 -0.15" rpy=" 0 0 3.14159"/>
-      <inertia ixx="100.0" ixy="0" ixz="0" iyy="100.0" iyz="0" izz="100.0" />
+      <inertia ixx="1.0" ixy="0" ixz="0" iyy="1.0" iyz="0" izz="1.0" />
     </inertial>
     <collision name='collision'>
@@ -26,5 +27,5 @@
     </visual>
     <collision name='caster1_collision'>
-      <origin xyz="0.45 0.22 -0.05" rpy=" 0 0 0"/>
+      <origin xyz="0.45 0 -0.05" rpy=" 0 0 0"/>
       <geometry>
         <sphere radius="0.05"/>
@@ -35,6 +36,6 @@
             <mu>0</mu>
             <mu2>0</mu2>
-            <slip1>5.0</slip1>
-            <slip2>5.0</slip2>
+            <slip1>1.0</slip1>
+            <slip2>1.0</slip2>
           </ode>
         </friction>
@@ -42,5 +43,5 @@
     </collision>
     <visual name='caster1_visual'>
-      <origin xyz="0.45 0.22 -0.05" rpy=" 0 0 0"/>
+      <origin xyz="0.45 0 -0.05" rpy=" 0 0 0"/>
       <geometry>
         <sphere radius="0.05"/>
@@ -48,5 +49,5 @@
     </visual>
     <collision name='caster2_collision'>
-      <origin xyz="0.45 -0.22 -0.05" rpy=" 0 0 0"/>
+      <origin xyz="-0.45 0 -0.05" rpy=" 0 0 0"/>
       <geometry>
         <sphere radius="0.05"/>
@@ -57,6 +58,6 @@
             <mu>0</mu>
             <mu2>0</mu2>
-            <slip1>5.0</slip1>
-            <slip2>5.0</slip2>
+            <slip1>1.0</slip1>
+            <slip2>1.0</slip2>
           </ode>
         </friction>
@@ -64,49 +65,5 @@
     </collision>
     <visual name='caster2_visual'>
-      <origin xyz="0.45 -0.22 -0.05" rpy=" 0 0 0"/>
-      <geometry>
-        <sphere radius="0.05"/>
-      </geometry>
-    </visual>
-    <collision name='caster3_collision'>
-      <origin xyz="-0.45 0.22 -0.05" rpy=" 0 0 0"/>
-      <geometry>
-        <sphere radius="0.05"/>
-      </geometry>
-      <surface>
-        <friction>
-          <ode>
-            <mu>0</mu>
-            <mu2>0</mu2>
-            <slip1>5.0</slip1>
-            <slip2>5.0</slip2>
-          </ode>
-        </friction>
-      </surface>
-    </collision>
-    <visual name='caster3_visual'>
-      <origin xyz="-0.45 0.22 -0.05" rpy=" 0 0 0"/>
-      <geometry>
-        <sphere radius="0.05"/>
-      </geometry>
-    </visual>
-    <collision name='caster4_collision'>
-      <origin xyz="-0.45 -0.22 -0.05" rpy=" 0 0 0"/>
-      <geometry>
-        <sphere radius="0.05"/>
-      </geometry>
-      <surface>
-        <friction>
-          <ode>
-            <mu>0</mu>
-            <mu2>0</mu2>
-            <slip1>5.0</slip1>
-            <slip2>5.0</slip2>
-          </ode>
-        </friction>
-      </surface>
-    </collision>
-    <visual name='caster4_visual'>
-      <origin xyz="-0.45 -0.22 -0.05" rpy=" 0 0 0"/>
+      <origin xyz="-0.45 0 -0.05" rpy=" 0 0 0"/>
       <geometry>
         <sphere radius="0.05"/>
@@ -120,19 +77,4 @@
         <cylinder radius="0.1" length="0.03"/>
       </geometry>
-      <surface>
-        <friction>
-          <ode>
-            <mu>50</mu>
-            <mu2>50</mu2>
-            <slip1>0</slip1>
-            <slip2>0</slip2>
-          </ode>
-        </friction>
-        <contact>
-          <ode>
-            <min_depth>10</min_depth>
-          </ode>
-        </contact>
-      </surface>
     </collision>
     <visual name="left_wheel_visual">
@@ -155,19 +97,4 @@
         <cylinder radius="0.1" length="0.03"/>
       </geometry>
-      <surface>
-        <friction>
-          <ode>
-            <mu>50</mu>
-            <mu2>50</mu2>
-            <slip1>0</slip1>
-            <slip2>0</slip2>
-          </ode>
-        </friction>
-        <contact>
-          <ode>
-            <min_depth>10</min_depth>
-          </ode>
-        </contact>
-      </surface>
     </collision>
     <visual name="right_wheel_visual">
@@ -190,6 +117,10 @@
     <material>WheelMaterial</material>
   </gazebo>
+  <joint name="base_link_to_chassis" type="fixed">
+    <parent link="base_link"/>
+    <child link="chassis"/>
+  </joint>
   <joint type="continuous" name="left_wheel_hinge">
-    <origin xyz="0 0.22 0" rpy="0 0 0"/>
+    <origin xyz="0 0.40 0" rpy="0 0 0"/>
     <child link="left_wheel"/>
     <parent link="chassis"/>
@@ -199,5 +130,5 @@
   </joint>
   <joint type="continuous" name="right_wheel_hinge">
-    <origin xyz="0 -0.22 0" rpy="0 0 0"/>
+    <origin xyz="0 -0.40 0" rpy="0 0 0"/>
     <child link="right_wheel"/>
     <parent link="chassis"/>
@@ -206,6 +137,6 @@
     <joint_properties damping="0.0" friction="0.0"/>
   </joint>
-  <sensor_d435 parent="chassis">
+  <xacro:sensor_d435 parent="chassis">
     <origin xyz="0.63 0 0" rpy="0 0 0"/>
-  </sensor_d435>
+  </xacro:sensor_d435>
 </robot>
